Commit message: 更好的抬升设计的双导轮方案

File: pkgs/robot_r2_description/urdf/robot_r2.urdf (robot description, URDF)
Before this commit: robot simple_chassis_robot, 22 links, 21 joints
Links:
- added link guide_support_ml2, mass 0.05; collision box size=0.020 0.020 0.170; visual box size=0.020 0.020 0.170
- added link guide_support_mr2, mass 0.05; collision box size=0.020 0.020 0.170; visual box size=0.020 0.020 0.170
- added link guide_wheel_ml2, mass 0.02; collision cylinder length=0.017 radius=0.019; visual cylinder length=0.017 radius=0.019
- added link guide_wheel_mr2, mass 0.02; collision cylinder length=0.017 radius=0.019; visual cylinder length=0.017 radius=0.019
Joints:
- added joint guide_support_ml2_joint: type fixed, parent base_link, child guide_support_ml2, origin xyz=0.080 0.224 -0.095 rpy=0 0 0
- added joint guide_support_mr2_joint: type fixed, parent base_link, child guide_support_mr2, origin xyz=0.080 -0.224 -0.095 rpy=0 0 0
- added joint guide_wheel_ml2_joint: type fixed, parent guide_support_ml2, child guide_wheel_ml2, origin xyz=0 0 -0.085 rpy=0 0 0
- added joint guide_wheel_mr2_joint: type fixed, parent guide_support_mr2, child guide_wheel_mr2, origin xyz=0 0 -0.085 rpy=0 0 0

Commit message: feature 加入加取kfs模型和控制器

File: pkgs/robot_r2_description/urdf/robot_r2.urdf (robot description, URDF)
Before this commit: robot simple_chassis_robot, 26 links, 25 joints
Links:
- added link bar_mount, mass 0.02; collision box size=0.010 0.010 0.010; visual box size=0.010 0.010 0.010
- added link gripper_left, mass 0.05; collision box size=0.10 0.01 0.20; visual box size=0.10 0.01 0.20
- added link gripper_right, mass 0.05; collision box size=0.10 0.01 0.20; visual box size=0.10 0.01 0.20
- added link long_bar, mass 0.16; collision box size=0.020 0.428 0.020; visual box size=0.020 0.428 0.020
Joints:
- added joint bar_mount_prismatic_joint: type prismatic, parent base_link, child bar_mount, origin xyz=0.2925 0 0.260 rpy=0 0 0, axis 0 0 1, limit lower=-0.180 upper=0.240 effort=100 velocity=0.2
- added joint gripper_left_joint: type prismatic, parent long_bar, child gripper_left, origin xyz=0.1175 0.209 0 rpy=0 0 0, axis 0 1 0, limit lower=-0.209 upper=0 effort=50 velocity=0.3
- added joint gripper_right_joint: type prismatic, parent long_bar, child gripper_right, origin xyz=0.1175 -0.209 0 rpy=0 0 0, axis 0 1 0, limit lower=0 upper=0.209 effort=50 velocity=0.3
- added joint long_bar_revolute_joint: type revolute, parent bar_mount, child long_bar, origin xyz=0 0 0 rpy=0 0 0, axis 0 1 0, limit lower=-3.14159 upper=0 effort=100 velocity=3.0

Commit message: feature 定点装载kfs

File: pkgs/robot_r2_description/urdf/robot_r2.urdf (robot description, URDF)
Before this commit: robot simple_chassis_robot, 30 links, 29 joints
Joints:
- joint gripper_left_joint: origin xyz=0.1175 0.209 0 rpy=0 0 0 -> xyz=0.1175 0.209 -0.030 rpy=0 0 0
- joint gripper_right_joint: origin xyz=0.1175 -0.209 0 rpy=0 0 0 -> xyz=0.1175 -0.209 -0.030 rpy=0 0 0

Commit message: feature 修改模型加入kfs锁定结构

File: pkgs/robot_r2_description/urdf/robot_r2.urdf (robot description, URDF)
Before this commit: robot simple_chassis_robot, 30 links, 29 joints
Links:
- added link vertical_bar_left, mass 0.2; collision box size=0.020 0.020 0.550; visual box size=0.020 0.020 0.550
- added link vertical_bar_rear, mass 0.2; collision box size=0.020 0.020 0.550; visual box size=0.020 0.020 0.550
- added link vertical_bar_right, mass 0.2; collision box size=0.020 0.020 0.550; visual box size=0.020 0.020 0.550
Joints:
- added joint vertical_bar_left_joint: type fixed, parent base_link, child vertical_bar_left, origin xyz=0 0.190 0.285 rpy=0 0 0
- added joint vertical_bar_rear_joint: type fixed, parent base_link, child vertical_bar_rear, origin xyz=-0.180 0 0.285 rpy=0 0 0
- added joint vertical_bar_right_joint: type fixed, parent base_link, child vertical_bar_right, origin xyz=0 -0.190 0.285 rpy=0 0 0

Commit message: feature 上台阶装载kfs

File: pkgs/robot_r2_description/urdf/robot_r2.urdf (robot description, URDF)
Before this commit: robot simple_chassis_robot, 33 links, 32 joints
Joints:
- joint vertical_bar_rear_joint: origin xyz=-0.180 0 0.285 rpy=0 0 0 -> xyz=-0.190 0 0.285 rpy=0 0 0

Commit message: feature 下台阶装载kfs

File: pkgs/robot_r2_description/urdf/robot_r2.urdf (robot description, URDF)
Before this commit: robot simple_chassis_robot, 33 links, 32 joints
Links:
- added link guide_support_fc, mass 0.05; collision box size=0.020 0.020 0.170; visual box size=0.020 0.020 0.170
Joints:
- added joint guide_support_fc_joint: type fixed, parent base_link, child guide_support_fc, origin xyz=0.340 0 -0.095 rpy=0 0 0

Commit message: recode 7.13 17:50

File: pkgs/robot_r2_description/urdf/robot_r2.urdf (robot description, URDF)
Before this commit: robot simple_chassis_robot, 34 links, 33 joints
Links:
- removed link bar_mount
- removed link long_bar
- added link gripper_extension, mass 0.08; visual box size=0.600 0.020 0.020
- added link gripper_lift, mass 0.02; collision box size=0.010 0.010 0.010; visual box size=0.010 0.010 0.010
- added link gripper_root, mass 0.16; collision box size=0.020 0.428 0.020; visual box size=0.020 0.428 0.020
- added link gripper_tip, mass 0.16; collision box size=0.020 0.428 0.020; visual box size=0.020 0.428 0.020
Joints:
- removed joint bar_mount_prismatic_joint
- removed joint long_bar_revolute_joint
- added joint gripper_extension_joint: type fixed, parent gripper_root, child gripper_extension, origin xyz=0 0 0 rpy=0 0 0
- added joint gripper_lift_joint: type prismatic, parent base_link, child gripper_lift, origin xyz=0.2925 0 0.260 rpy=0 0 0, axis 0 0 1, limit lower=-0.180 upper=0.240 effort=100 velocity=0.2
- added joint gripper_root_joint: type revolute, parent gripper_lift, child gripper_root, origin xyz=0 0 0 rpy=0 0 0, axis 0 1 0, limit lower=-1.5708 upper=0 effort=100 velocity=3.0
- added joint gripper_tip_joint: type revolute, parent gripper_extension, child gripper_tip, origin xyz=0.600 0 0 rpy=0 0 0, axis 0 1 0, limit lower=-1.5708 upper=1.5708 effort=100 velocity=3.0
- joint gripper_left_joint: origin xyz=0.1175 0.209 -0.030 rpy=0 0 0 -> xyz=0.060 0.209 -0.030 rpy=0 0 0; parent long_bar -> gripper_tip
- joint gripper_right_joint: origin xyz=0.1175 -0.209 -0.030 rpy=0 0 0 -> xyz=0.060 -0.209 -0.030 rpy=0 0 0; parent long_bar -> gripper_tip

Commit message: recode 7.18 16:04

File: pkgs/robot_r2_description/urdf/robot_r2.urdf (robot description, URDF)
Before this commit: robot simple_chassis_robot, 36 links, 35 joints
Links:
- removed link gripper_lift
- added link kfs_lift_plate, mass 0.5; collision box size=0.400 0.350 0.010; visual box size=0.400 0.350 0.010
- link gripper_extension: geometry collision box size=0.530 0.020 0.020; visual box size=0.530 0.020 0.020
Joints:
- removed joint gripper_lift_joint
- added joint kfs_lift_joint: type prismatic, parent base_link, child kfs_lift_plate, origin xyz=0.0975 0 0.015 rpy=0 0 0, axis 0 0 1, limit lower=0.0 upper=0.42 effort=1000 velocity=0.2
- joint gripper_root_joint: limit lower=-1.5708 upper=0 effort=100 velocity=3.0 -> lower=-1.5707963267948966 upper=0.7853981633974483 effort=100 velocity=3.0; origin xyz=0 0 0 rpy=0 0 0 -> xyz=0.30 0 0.060 rpy=0 0 0; parent gripper_lift -> base_link
- joint gripper_tip_joint: origin xyz=0.600 0 0 rpy=0 0 0 -> xyz=0.530 0 0 rpy=0 0 0
- joint vertical_bar_left_joint: origin xyz=0 0.190 0.285 rpy=0 0 0 -> xyz=0.100 0.190 0.285 rpy=0 0 0
- joint vertical_bar_rear_joint: origin xyz=-0.190 0 0.285 rpy=0 0 0 -> xyz=-0.115 0 0.285 rpy=0 0 0
- joint vertical_bar_right_joint: origin xyz=0 -0.190 0.285 rpy=0 0 0 -> xyz=0.100 -0.190 0.285 rpy=0 0 0

Commit message: feature 阶段2.1和2.2

File: pkgs/robot_r2_description/urdf/robot_r2.urdf (robot description, URDF)
Before this commit: robot simple_chassis_robot, 36 links, 35 joints
Joints:
- joint vertical_bar_rear_joint: origin xyz=-0.115 0 0.285 rpy=0 0 0 -> xyz=-0.130 0 0.285 rpy=0 0 0
