Commit message: recode 8.1 22:28

File: src/robot_r2_description/urdf/robot_r2.urdf (robot description, URDF)
Before this commit: robot simple_chassis_robot, 36 links, 35 joints
Joints:
- joint gripper_left_joint: limit lower=-0.209 upper=0 effort=50 velocity=0.3 -> lower=0 upper=0.209 effort=50 velocity=0.3; origin xyz=0.060 0.209 -0.030 rpy=0 0 0 -> xyz=0.060 0 -0.030 rpy=0 0 0
- joint gripper_right_joint: axis 0 1 0 -> 0 -1 0; origin xyz=0.060 -0.209 -0.030 rpy=0 0 0 -> xyz=0.060 0 -0.030 rpy=0 0 0
- joint gripper_root_joint: limit lower=-1.5707963267948966 upper=0.7853981633974483 effort=100 velocity=3.0 -> lower=0.0 upper=2.356194490192345 effort=100 velocity=3.0; origin xyz=0.30 0 0.060 rpy=0 0 0 -> xyz=0.30 0 0.060 rpy=0 -1.5707963267948966 0
- joint gripper_tip_joint: axis 0 1 0 -> 0 -1 0; limit lower=-1.5708 upper=1.5708 effort=100 velocity=3.0 -> lower=0.0 upper=3.141592653589793 effort=100 velocity=3.0; origin xyz=0.530 0 0 rpy=0 0 0 -> xyz=0.530 0 0 rpy=0 1.5707963267948966 0

Commit message: refactor kfs load

File: src/robot_r2_description/urdf/robot_r2.urdf (robot description, URDF)
Before this commit: robot simple_chassis_robot, 36 links, 35 joints
Joints:
- joint gripper_root_joint: limit lower=0.0 upper=2.356194490192345 effort=100 velocity=3.0 -> lower=-0.2617993877991494 upper=2.356194490192345 effort=100 velocity=3.0
